Commit message: its win

File: src/tinker_description/urdf/tinker_urdf.urdf (robot description, URDF)
Before this commit: robot tinker_urdf, 11 links, 10 joints
Links:
- link base_link: geometry collision mesh filename=file:///home/none/Challenge-Tinker/src/tinker_description/m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; visual mesh filename=file:///home/none/Challenge-Tinker/src/tinker_description/m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
- link link_l_ankle: geometry collision cylinder length=0.13 radius=0.015; visual mesh filename=file:///home/none/Challenge-Tinker/src/tinker_description/m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
- link link_l_knee: geometry visual mesh filename=file:///home/none/Challenge-Tinker/src/tinker_description/m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
- link link_l_pitch: geometry collision mesh filename=file:///home/none/Challenge-Tinker/src/tinker_description/m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; visual mesh filename=file:///home/none/Challenge-Tinker/src/tinker_description/m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
- link link_l_roll: geometry visual mesh filename=file:///home/none/Challenge-Tinker/src/tinker_description/m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
- link link_l_yaw: geometry visual mesh filename=file:///home/none/Challenge-Tinker/src/tinker_description/m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
- link link_r_ankle: geometry collision cylinder length=0.13 radius=0.015; visual mesh filename=file:///home/none/Challenge-Tinker/src/tinker_description/m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
- link link_r_knee: geometry visual mesh filename=file:///home/none/Challenge-Tinker/src/tinker_description/m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
- link link_r_pitch: geometry collision mesh filename=file:///home/none/Challenge-Tinker/src/tinker_description/m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; visual mesh filename=file:///home/none/Challenge-Tinker/src/tinker_description/m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
- link link_r_roll: geometry visual mesh filename=file:///home/none/Challenge-Tinker/src/tinker_description/m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
- link link_r_yaw: geometry visual mesh filename=file:///home/none/Challenge-Tinker/src/tinker_description/m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
